File: power-meter-pcb/strain-gauge-amplifier.kicad_sch (KiCad schematic)
At the start: 20 parts, among them J5 Side A, J6 Side B, Q3 AS2302, U7 ADS1232IPW

Commit message: Tidying schematic
Other:
- moved on the sheet: C15
Changed lines of the file:
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@@
 		(stroke
 			(width 0)
-			(type default)
+			(type dot)
 		)
 	)
@@
 		(stroke
 			(width 0)
-			(type default)
+			(type dot)
 		)
 	)
@@
 		(stroke
 			(width 0)
-			(type default)
+			(type dot)
 		)
 	)
@@
 		(stroke
 			(width 0)
-			(type default)
+			(type dot)
 		)
 	)
@@
 		(stroke
 			(width 0)
-			(type default)
+			(type dot)
 		)
 	)
@@
 		(stroke
 			(width 0)
-			(type default)
+			(type dot)
 		)
 	)
@@
 		(stroke
 			(width 0)
-			(type default)
+			(type dot)
 		)
 	)
@@
 		(stroke
 			(width 0)
-			(type default)
+			(type dot)
 		)
 	)
@@
 		(stroke
 			(width 0)
-			(type default)
+			(type dot)
 		)
 	)
@@
 		(stroke
 			(width 0)
-			(type default)
+			(type dot)
 		)
 	)
@@
 		(stroke
 			(width 0)
-			(type default)
+			(type dot)
 		)
 	)
@@
 		(stroke
 			(width 0)
-			(type default)
+			(type dot)
 		)
 	)
@@
 		(stroke
 			(width 0)
-			(type default)
+			(type dot)
 		)
 	)
@@
 	(wire
 		(pts
-			(xy 234.95 95.25) (xy 234.95 97.79)
+			(xy 236.22 95.25) (xy 236.22 97.79)
 		)
 		(stroke
@@
 		(stroke
 			(width 0)
-			(type default)
+			(type dot)
 		)
 	)
@@
 		(stroke
 			(width 0)
-			(type default)
+			(type dot)
 		)
 	)
@@
 		(stroke
 			(width 0)
-			(type default)
+			(type dot)
 		)
 	)
@@
 		(stroke
 			(width 0)
-			(type default)
+			(type dot)
 		)
 	)
@@
 		(stroke
 			(width 0)
-			(type default)
+			(type dot)
 		)
 	)
@@
 		(stroke
 			(width 0)
-			(type default)
+			(type dot)
 		)
 	)
@@
 		(stroke
 			(width 0)
-			(type default)
+			(type dot)
 		)
 	)
@@
 		(stroke
 			(width 0)
-			(type default)
+			(type dot)
 		)
 	)
@@
 	(wire
 		(pts
-			(xy 234.95 85.09) (xy 234.95 87.63)
+			(xy 236.22 85.09) (xy 236.22 87.63)
 		)
 		(stroke
@@
 		(stroke
 			(width 0)
-			(type default)
+			(type dot)
 		)
 	)
@@
 		(stroke
 			(width 0)
-			(type default)
+			(type dot)
 		)
 	)
@@
 		(stroke
 			(width 0)
-			(type default)
+			(type dot)
 		)
 	)
@@
 			(width 0)
 			(type default)
+		)
+	)
+	(text_box "Strain gauges (SG1, SG2, SG3 and SG4) are mounted off-board."
+		(exclude_from_sim no)
+		(at 31.75 97.79 0)
+		(size 30.48 8.89)
+		(stroke
+			(width 0)
+			(type default)
+		)
+		(fill
+			(type none)
+		)
+		(effects
+			(font
+				(size 1.27 1.27)
+			)
+			(justify left top)
 		)
 	)
@@
 	(symbol
 		(lib_id "Device:C")
-		(at 234.95 91.44 0)
+		(at 236.22 91.44 0)
 		(unit 1)
 		(exclude_from_sim no)
@@
 		(fields_autoplaced yes)
 		(property "Reference" "C15"
-			(at 238.76 90.1699 0)
+			(at 240.03 90.1699 0)
 			(effects
 				(font
@@
 		)
 		(property "Value" "0.1u"
-			(at 238.76 92.7099 0)
+			(at 240.03 92.7099 0)
 			(effects
 				(font
@@
 		)
 		(property "Footprint" "Capacitor_SMD:C_0603_1608Metric_Pad1.08x0.95mm_HandSolder"
-			(at 235.9152 95.25 0)
+			(at 237.1852 95.25 0)
 			(effects
 				(font
@@
 		)
 		(property "Datasheet" "~"
-			(at 234.95 91.44 0)
+			(at 236.22 91.44 0)
 			(effects
 				(font
@@
 		)
 		(property "Description" "Unpolarized capacitor"
-			(at 234.95 91.44 0)
+			(at 236.22 91.44 0)
 			(effects
 				(font
@@
 	(symbol
 		(lib_id "power:GNDD")
-		(at 234.95 97.79 0)
+		(at 236.22 97.79 0)
 		(unit 1)
 		(exclude_from_sim no)
@@
 		(fields_autoplaced yes)
 		(property "Reference" "#PWR041"
-			(at 234.95 104.14 0)
+			(at 236.22 104.14 0)
 			(effects
 				(font
@@
 		)
 		(property "Value" "GNDD"
-			(at 234.95 101.6 0)
+			(at 236.22 101.6 0)
 			(effects
 				(font
@@
 		)
 		(property "Footprint" ""
-			(at 234.95 97.79 0)
+			(at 236.22 97.79 0)
 			(effects
 				(font
@@
 		)
 		(property "Datasheet" ""
-			(at 234.95 97.79 0)
+			(at 236.22 97.79 0)
 			(effects
 				(font
@@
 		)
 		(property "Description" "Power symbol creates a global label with name \"GNDD\" , digital ground"
-			(at 234.95 97.79 0)
+			(at 236.22 97.79 0)
 			(effects
 				(font
@@
 	(symbol
 		(lib_id "power:+3.3V")
-		(at 234.95 85.09 0)
+		(at 236.22 85.09 0)
 		(unit 1)
 		(exclude_from_sim no)
@@
 		(fields_autoplaced yes)
 		(property "Reference" "#PWR040"
-			(at 234.95 88.9 0)
+			(at 236.22 88.9 0)
 			(effects
 				(font
@@
 		)
 		(property "Value" "+3.3V"
-			(at 234.95 80.01 0)
+			(at 236.22 80.01 0)
 			(effects
 				(font
@@
 		)
 		(property "Footprint" ""
-			(at 234.95 85.09 0)
+			(at 236.22 85.09 0)
 			(effects
 				(font
@@
 		)
 		(property "Datasheet" ""
-			(at 234.95 85.09 0)
+			(at 236.22 85.09 0)
 			(effects
 				(font
@@
 		)
 		(property "Description" "Power symbol creates a global label with name \"+3.3V\""
-			(at 234.95 85.09 0)
-			(effects
-				(font
+			(at 236.22 85.09 0)
+			(effects
+				(font

Commit message: Improved board outline, in the middle of layout changes
Parts:
- renumbered R16 to R17, R17 to R18, R18 to R19, R19 to R20
Changed lines of the file:
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@@
 		(dnp no)
 		(fields_autoplaced yes)
-		(property "Reference" "#PWR037"
+		(property "Reference" "#PWR038"
 			(at 161.29 71.12 0)
 			(effects
@@
 			(project "power-meter-pcb"
 				(path "/73d1dc3f-3725-4767-8c11-2d32e15ee0d6/feb88761-b4a9-421c-bc5f-37e5e311e229"
-					(reference "#PWR037")
+					(reference "#PWR038")
 					(unit 1)
 				)
@@
 		(dnp no)
 		(fields_autoplaced yes)
-		(property "Reference" "#PWR035"
+		(property "Reference" "#PWR036"
 			(at 151.13 139.7 0)
 			(effects
@@
 			(project "power-meter-pcb"
 				(path "/73d1dc3f-3725-4767-8c11-2d32e15ee0d6/feb88761-b4a9-421c-bc5f-37e5e311e229"
-					(reference "#PWR035")
+					(reference "#PWR036")
 					(unit 1)
 				)
@@
 		(dnp no)
 		(fields_autoplaced yes)
-		(property "Reference" "#PWR038"
+		(property "Reference" "#PWR039"
 			(at 224.79 88.9 0)
 			(effects
@@
 			(project "power-meter-pcb"
 				(path "/73d1dc3f-3725-4767-8c11-2d32e15ee0d6/feb88761-b4a9-421c-bc5f-37e5e311e229"
-					(reference "#PWR038")
+					(reference "#PWR039")
 					(unit 1)
 				)
@@
 		(dnp no)
 		(fields_autoplaced yes)
-		(property "Reference" "R17"
+		(property "Reference" "R18"
 			(at 185.42 81.28 90)
 			(effects
@@
 			(project "power-meter-pcb"
 				(path "/73d1dc3f-3725-4767-8c11-2d32e15ee0d6/feb88761-b4a9-421c-bc5f-37e5e311e229"
-					(reference "R17")
+					(reference "R18")
 					(unit 1)
 				)
@@
 		(on_board yes)
 		(dnp no)
-		(property "Reference" "R19"
+		(property "Reference" "R20"
 			(at 185.42 100.584 90)
 			(effects
@@
 			(project "power-meter-pcb"
 				(path "/73d1dc3f-3725-4767-8c11-2d32e15ee0d6/feb88761-b4a9-421c-bc5f-37e5e311e229"
-					(reference "R19")
+					(reference "R20")
 					(unit 1)
 				)
@@
 		(dnp no)
 		(fields_autoplaced yes)
-		(property "Reference" "R16"
+		(property "Reference" "R17"
 			(at 59.69 111.76 90)
 			(effects
@@
 			(project "power-meter-pcb"
 				(path "/73d1dc3f-3725-4767-8c11-2d32e15ee0d6/feb88761-b4a9-421c-bc5f-37e5e311e229"
-					(reference "R16")
+					(reference "R17")
 					(unit 1)
 				)
@@
 		(dnp no)
 		(fields_autoplaced yes)
-		(property "Reference" "#PWR034"
+		(property "Reference" "#PWR035"
 			(at 151.13 62.23 0)
 			(effects
@@
 			(project "power-meter-pcb"
 				(path "/73d1dc3f-3725-4767-8c11-2d32e15ee0d6/feb88761-b4a9-421c-bc5f-37e5e311e229"
-					(reference "#PWR034")
+					(reference "#PWR035")
 					(unit 1)
 				)
@@
 		(dnp no)
 		(fields_autoplaced yes)
-		(property "Reference" "#PWR039"
+		(property "Reference" "#PWR040"
 			(at 224.79 104.14 0)
 			(effects
@@
 			(project "power-meter-pcb"
 				(path "/73d1dc3f-3725-4767-8c11-2d32e15ee0d6/feb88761-b4a9-421c-bc5f-37e5e311e229"
-					(reference "#PWR039")
+					(reference "#PWR040")
 					(unit 1)
 				)
@@
 		(dnp no)
 		(fields_autoplaced yes)
-		(property "Reference" "#PWR041"
+		(property "Reference" "#PWR042"
 			(at 236.22 104.14 0)
 			(effects
@@
 			(project "power-meter-pcb"
 				(path "/73d1dc3f-3725-4767-8c11-2d32e15ee0d6/feb88761-b4a9-421c-bc5f-37e5e311e229"
-					(reference "#PWR041")
+					(reference "#PWR042")
 					(unit 1)
 				)
@@
 		(dnp no)
 		(fields_autoplaced yes)
-		(property "Reference" "#PWR040"
+		(property "Reference" "#PWR041"
 			(at 236.22 88.9 0)
 			(effects
@@
 			(project "power-meter-pcb"
 				(path "/73d1dc3f-3725-4767-8c11-2d32e15ee0d6/feb88761-b4a9-421c-bc5f-37e5e311e229"
-					(reference "#PWR040")
+					(reference "#PWR041")
 					(unit 1)
 				)
@@
 		(on_board yes)
 		(dnp no)
-		(property "Reference" "R18"
+		(property "Reference" "R19"
 			(at 185.42 92.964 90)
 			(effects
@@
 			(project "power-meter-pcb"
 				(path "/73d1dc3f-3725-4767-8c11-2d32e15ee0d6/feb88761-b4a9-421c-bc5f-37e5e311e229"
-					(reference "R18")
+					(reference "R19")
 					(unit 1)
 				)
@@
 		(dnp no)
 		(fields_autoplaced yes)
-		(property "Reference" "#PWR036"
+		(property "Reference" "#PWR037"
 			(at 158.75 139.7 0)
 			(effects
@@
 			(project "power-meter-pcb"
 				(path "/73d1dc3f-3725-4767-8c11-2d32e15ee0d6/feb88761-b4a9-421c-bc5f-37e5e311e229"
-					(reference "#PWR036")
-					(unit 1)
-				)
+					(reference "#PWR037")
+					(unit 1)
+				)

Commit message: Layout almost done, but will likely swap to a 4 layer PCB
Parts:
- removed NT1: NetTie_2, NetTie:NetTie-2_SMD_Pad0.5mm, symbol Device:NetTie_2
Connections:
- net GP is gone; now on net +3.3VA: U7.16 (REFP)
- no-connect marks 0 -> 1
Changed lines of the file:
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@@
 		(date "2024-04-18")
 		(company "Monash Human Power - Jotham Gates & Oscar Varney")
+		(comment 1 "For the secondary crank, set J3 to short pins 2 and 3 and short J1 and J2.")
 	)
 	(junction
@@
 		(color 0 0 0 0)
 	)
+	(no_connect
+		(at 173.99 100.33)
+	)
 	(bus_entry
 		(at 203.2 87.63)
@@
 	(wire
 		(pts
-			(xy 129.54 63.5) (xy 135.89 63.5)
-		)
-		(stroke
-			(width 0)
-			(type default)
-		)
-	)
-	(wire
-		(pts
 			(xy 88.9 76.2) (xy 91.44 76.2)
 		)
@@
 	(wire
 		(pts
-			(xy 88.9 63.5) (xy 124.46 63.5)
+			(xy 88.9 63.5) (xy 135.89 63.5)
 		)
 		(stroke
@@
 			)
 			(justify left top)
-		)
-	)
-	(label "GP"
-		(at 135.89 80.01 0)
-		(fields_autoplaced yes)
-		(effects
-			(font
-				(size 1.27 1.27)
-			)
-			(justify left bottom)
 		)
 	)
@@
 					(unit 1)
 				)
-			)
-		)
-	)
-	(symbol
-		(lib_id "Device:NetTie_2")
-		(at 127 63.5 0)
-		(unit 1)
-		(exclude_from_sim no)
-		(in_bom no)
-		(on_board yes)
-		(dnp no)
-		(property "Reference" "NT1"
-			(at 127 65.786 0)
-			(effects
-				(font
-					(size 1.27 1.27)
-				)
-			)
-		)
-		(property "Value" "NetTie_2"
-			(at 127 60.96 0)
-			(effects
-				(font
-					(size 1.27 1.27)
-				)
-				(hide yes)
-			)
-		)
-		(property "Footprint" "NetTie:NetTie-2_SMD_Pad0.5mm"
-			(at 127 63.5 0)
-			(effects
-				(font
-					(size 1.27 1.27)
-				)
-				(hide yes)
-			)
-		)
-		(property "Datasheet" "~"
-			(at 127 63.5 0)
-			(effects
-				(font
-					(size 1.27 1.27)
-				)
-				(hide yes)
-			)
-		)
-		(property "Description" "Net tie, 2 pins"
-			(at 127 63.5 0)
-			(effects
-				(font
-					(size 1.27 1.27)
-				)
-				(hide yes)
-			)
-		)
-		(pin "1"
-		)
-		(pin "2"
-		)
-		(instances
-			(project "power-meter-pcb"
-				(path "/73d1dc3f-3725-4767-8c11-2d32e15ee0d6/feb88761-b4a9-421c-bc5f-37e5e311e229"
-					(reference "NT1")
-					(unit 1)
-				)
