File: power-meter-pcb/accelerometer.kicad_sch (KiCad schematic)
At the start: 2 parts

Commit message: Re-centred schematics, added header for spare GPIO pins, touched up logos
Other:
- moved on the sheet: C16, MT1

Commit message: Added LED driven by temp sensor, updated numbering
Parts:
- renumbered C16 to C13
Changed lines of the file:
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@@
 	(title_block
 		(title "Cycling power meter FYP - Accelerometer and gyroscope")
-		(date "2024-07-05")
-		(rev "V1.0.2")
+		(date "2024-07-11")
+		(rev "V1.0.3")
 		(company "Monash Human Power - Jotham Gates & Oscar Varney")
 	)
@@
 			)
 		)
+		(property "Sim.Device" ""
+			(at 143.51 92.71 0)
+			(effects
+				(font
+					(size 1.27 1.27)
+				)
+				(hide yes)
+			)
+		)
+		(property "Sim.Pins" ""
+			(at 143.51 92.71 0)
+			(effects
+				(font
+					(size 1.27 1.27)
+				)
+				(hide yes)
+			)
+		)
 		(pin "4"
 		)
@@
 		(dnp no)
 		(fields_autoplaced yes)
-		(property "Reference" "#PWR047"
+		(property "Reference" "#PWR041"
 			(at 196.85 107.95 0)
 			(effects
@@
 			(project "power-meter-pcb"
 				(path "/73d1dc3f-3725-4767-8c11-2d32e15ee0d6/2b9cb85e-d958-4741-88c2-27e776d7a0b9"
-					(reference "#PWR047")
+					(reference "#PWR041")
 					(unit 1)
 				)
@@
 		(dnp no)
 		(fields_autoplaced yes)
-		(property "Reference" "#PWR046"
+		(property "Reference" "#PWR040"
 			(at 196.85 92.71 0)
 			(effects
@@
 			(project "power-meter-pcb"
 				(path "/73d1dc3f-3725-4767-8c11-2d32e15ee0d6/2b9cb85e-d958-4741-88c2-27e776d7a0b9"
-					(reference "#PWR046")
+					(reference "#PWR040")
 					(unit 1)
 				)
@@
 		(dnp no)
 		(fields_autoplaced yes)
-		(property "Reference" "#PWR045"
+		(property "Reference" "#PWR039"
 			(at 171.45 119.38 0)
 			(effects
@@
 			(project "power-meter-pcb"
 				(path "/73d1dc3f-3725-4767-8c11-2d32e15ee0d6/2b9cb85e-d958-4741-88c2-27e776d7a0b9"
-					(reference "#PWR045")
+					(reference "#PWR039")
 					(unit 1)
 				)
@@
 		(dnp no)
 		(fields_autoplaced yes)
-		(property "Reference" "#PWR044"
+		(property "Reference" "#PWR038"
 			(at 171.45 83.82 0)
 			(effects
@@
 			(project "power-meter-pcb"
 				(path "/73d1dc3f-3725-4767-8c11-2d32e15ee0d6/2b9cb85e-d958-4741-88c2-27e776d7a0b9"
-					(reference "#PWR044")
+					(reference "#PWR038")
 					(unit 1)
 				)
@@
 		(dnp no)
 		(fields_autoplaced yes)
-		(property "Reference" "C16"
+		(property "Reference" "C13"
 			(at 200.66 93.9799 0)
 			(effects
@@
 		)
 		(property "PlaceOnSecondary" "No"
+			(at 196.85 95.25 0)
+			(effects
+				(font
+					(size 1.27 1.27)
+				)
+				(hide yes)
+			)
+		)
+		(property "Sim.Device" ""
+			(at 196.85 95.25 0)
+			(effects
+				(font
+					(size 1.27 1.27)
+				)
+				(hide yes)
+			)
+		)
+		(property "Sim.Pins" ""
 			(at 196.85 95.25 0)
 			(effects
@@
 			(project "power-meter-pcb"
 				(path "/73d1dc3f-3725-4767-8c11-2d32e15ee0d6/2b9cb85e-d958-4741-88c2-27e776d7a0b9"
-					(reference "C16")
+					(reference "C13")
 					(unit 1)
 				)
@@
 		(dnp no)
 		(fields_autoplaced yes)
-		(property "Reference" "#PWR043"
+		(property "Reference" "#PWR037"
 			(at 100.33 96.52 0)
 			(effects
@@
 			(project "power-meter-pcb"
 				(path "/73d1dc3f-3725-4767-8c11-2d32e15ee0d6/2b9cb85e-d958-4741-88c2-27e776d7a0b9"
-					(reference "#PWR043")
+					(reference "#PWR037")
 					(unit 1)
 				)

Commit message: Fixed SPI pin labels
Connections:
- net SPI.SDI: now also MT1.1 (AP_SDO/AP_AD0); no longer MT1.14 (AP_SDA/AP_SDIO/AP_SDI)
- net SPI.SDO: now also MT1.14 (AP_SDA/AP_SDIO/AP_SDI); no longer MT1.1 (AP_SDO/AP_AD0)
Changed lines of the file:
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@@
 		)
 	)
-	(label "SPI.SDO"
+	(label "SPI.SDI"
 		(at 107.95 100.33 0)
 		(fields_autoplaced yes)
@@
 		)
 	)
-	(label "SPI.SDI"
+	(label "SPI.SDO"
 		(at 107.95 97.79 0)
 		(fields_autoplaced yes)
