File: power-meter-pcb/accelerometer.kicad_sch (KiCad schematic)
At the start: 2 parts

Commit message: Sorting out parts to order and component changes
Parts:
- C13, MT1: SchematicVersionModified (none) -> V1.0.4
Changed lines of the file:
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@@
+			)
+		)
+		(property "SchematicVersionModified" "V1.0.4"
+			(at 143.51 92.71 0)
+			(effects
+				(font
+					(size 1.27 1.27)
+				)
+				(hide yes)
 			)
 		)
@@
 			(at 196.85 95.25 0)
 			(effects
+				(font
+					(size 1.27 1.27)
+				)
+				(hide yes)
+			)
+		)
+		(property "SchematicVersionModified" "V1.0.4"
+			(at 196.85 95.25 0)
+			(effects
